Commit message: created lidar and intrinsics. updated launch file to spawn robot within gazebo world. created test world for lidar object feedback

File: src/robot_core/src/robot_description/robot_core.urdf (robot description, URDF)
Before this commit: robot icarus, 2 links, 1 joints
Links:
- added link lidar_link, mass .17; collision cylinder length=.06 radius=${lidar_radius}; visual cylinder length=.06 radius=${lidar_radius}
Joints:
- added joint lidar_joint: type fixed, parent base_link, child lidar_link, origin xyz=${-chassis_length/2 + lidar_radius} 0 ${chassis_height/2+.02} rpy=0 0 0
